Commit message: migrated to ros2 and changed limits

File: arm.urdf (robot description, URDF)
Before this commit: robot servoarm, 8 links, 7 joints
Joints:
- joint joint1: limit lower=1.56 upper=4.68 effort=1000.0 velocity=1.0 -> lower=-1.57 upper=1.57 effort=1000.0 velocity=1.0
- joint joint2: limit lower=0.0 upper=3.12 effort=1000.0 velocity=1.0 -> lower=0 upper=1.57 effort=1000.0 velocity=1.0
- joint joint3: limit lower=-1.7 upper=1.7 effort=1000.0 velocity=1.0 -> lower=-1.57 upper=1.57 effort=1000.0 velocity=1.0
- joint joint4: limit lower=-1.7 upper=1.7 effort=1000.0 velocity=1.0 -> lower=-1.57 upper=1.57 effort=1000.0 velocity=1.0
- joint joint5: limit lower=-3.17 upper=0.0 effort=1000.0 velocity=1.0 -> lower=-1.57 upper=1.57 effort=1000.0 velocity=1.0

Commit message: fixed joint2 direction

File: arm.urdf (robot description, URDF)
Before this commit: robot servoarm, 8 links, 7 joints
Joints:
- joint joint2: limit lower=0 upper=1.57 effort=1000.0 velocity=1.0 -> lower=-1.57 upper=0 effort=1000.0 velocity=1.0; origin xyz=0 0.19 0.28 -> xyz=0 0.19 0.28 rpy=1.57 0 0
